File: UINIO-DAP-Link.kicad_pcb (KiCad board)
At the start: 2 copper layers, 90.4 x 31 mm, 45 parts, among them J1 扩展板串口 & 电源输出, J2 扩展板 JTAG 输出, J3 JTAG_nTRST 跳线选择, J4 3.3V 跳线选择, J5 扩展板 SWD 输入, J6 DAPLink 固件下载接口, J7 JTAG/SWD 下载接口, U1 ME6211, U2 STM32F103C8T6, Y1 Crystal_GND24

Commit message: Release UINIO-DAP-Link 1.0.0.
Parts:
- moved ? 0.22 mm to (171.6, 107.2)
Other:
- outline, holes or cut-outs redrawn
Changed lines of the file:
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@@
   )
   (footprint "LOGO" (layer "B.Cu")
-    (at 171.34 107.17 -90)
+    (at 171.56 107.19 -90)
     (attr board_only exclude_from_pos_files exclude_from_bom)
     (fp_text reference "" (at 0 0 90) (layer "B.SilkS")
@@
   (gr_line (start 137.895 113.86) (end 142.945 113.86) (layer "B.SilkS") (width 0.1))
   (gr_line (start 188.92 92.874517) (end 188.92 121.774517) (layer "B.SilkS") (width 0.1))
-  (gr_line (start 144.52 102.05) (end 151.62 102.05) (layer "Edge.Cuts") (width 0.1))
+  (gr_line (start 144.52 101.75) (end 151.62 101.75) (layer "Edge.Cuts") (width 0.1))
   (gr_arc (start 102.68 98.06) (mid 102.987286 97.386407) (end 103.67 97.1) (layer "Edge.Cuts") (width 0.1))
   (gr_line (start 193.084 93.52) (end 193.084 121.27) (layer "Edge.Cuts") (width 0.1))
-  (gr_line (start 144.52 106.61) (end 144.52 102.05) (layer "Edge.Cuts") (width 0.1))
+  (gr_line (start 144.52 106.61) (end 144.52 101.75) (layer "Edge.Cuts") (width 0.1))
   (gr_line (start 103.67 117.7) (end 143.47 117.7) (layer "Edge.Cuts") (width 0.1))
   (gr_arc (start 143.42 97.1) (mid 144.195891 97.358999) (end 144.52 98.11) (layer "Edge.Cuts") (width 0.1))
-  (gr_line (start 151.62 100.48) (end 151.62 93.499) (layer "Edge.Cuts") (width 0.1))
+  (gr_line (start 151.62 100.18) (end 151.62 93.499) (layer "Edge.Cuts") (width 0.1))
   (gr_line (start 144.52 108.18) (end 151.62 108.18) (layer "Edge.Cuts") (width 0.1))
   (gr_arc (start 191.41 91.884) (mid 192.606648 92.33402) (end 193.084 93.52) (layer "Edge.Cuts") (width 0.1))
@@
   (gr_arc (start 193.084 121.27) (mid 192.531165 122.385345) (end 191.37 122.834) (layer "Edge.Cuts") (width 0.1))
   (gr_line (start 144.52 108.18) (end 144.52 113.05) (layer "Edge.Cuts") (width 0.1))
-  (gr_line (start 144.52 98.11) (end 144.52 100.48) (layer "Edge.Cuts") (width 0.1))
+  (gr_line (start 144.52 98.11) (end 144.52 100.18) (layer "Edge.Cuts") (width 0.1))
   (gr_line (start 153.41 91.884) (end 191.41 91.884) (layer "Edge.Cuts") (width 0.1))
   (gr_line (start 151.62 114.62) (end 151.62 121.249) (layer "Edge.Cuts") (width 0.1))
   (gr_arc (start 103.67 117.7) (mid 102.981443 117.426697) (end 102.68 116.75) (layer "Edge.Cuts") (width 0.1))
   (gr_line (start 151.62 113.05) (end 144.52 113.05) (layer "Edge.Cuts") (width 0.1))
-  (gr_line (start 144.52 100.48) (end 151.62 100.48) (layer "Edge.Cuts") (width 0.1))
+  (gr_line (start 144.52 100.18) (end 151.62 100.18) (layer "Edge.Cuts") (width 0.1))
   (gr_line (start 144.52 116.61) (end 144.52 114.62) (layer "Edge.Cuts") (width 0.1))
   (gr_line (start 103.67 97.1) (end 143.42 97.1) (layer "Edge.Cuts") (width 0.1))
@@
   (gr_line (start 102.68 98.06) (end 102.68 116.75) (layer "Edge.Cuts") (width 0.1))
   (gr_line (start 151.62 106.61) (end 144.52 106.61) (layer "Edge.Cuts") (width 0.1))
-  (gr_line (start 151.62 106.61) (end 151.62 102.05) (layer "Edge.Cuts") (width 0.1))
+  (gr_line (start 151.62 106.61) (end 151.62 101.75) (layer "Edge.Cuts") (width 0.1))
   (gr_arc (start 151.62 93.499) (mid 152.184916 92.325666) (end 153.41 91.884) (layer "Edge.Cuts") (width 0.1))
   (gr_line (start 144.52 98.11) (end 144.52 116.61) (layer "User.1") (width 0.1))
@@
   (gr_line (start 151.62 93.499) (end 151.62 121.249) (layer "User.1") (width 0.1))
   (gr_rect (start 102.68 97.1) (end 144.52 117.7) (layer "User.1") (width 0.1) (fill none))
+  (gr_rect (start 143.44 97.1) (end 146.88 100.18) (layer "User.1") (width 0.1) (fill none))
+  (gr_rect (start 144.58 114.62) (end 148.02 117.7) (layer "User.1") (width 0.1) (fill none))
   (gr_rect (start 149.26 113.05) (end 150.91 114.62) (layer "User.1") (width 0.1) (fill none))
   (gr_rect (start 151.62 91.88) (end 193.088 122.834) (layer "User.1") (width 0.1) (fill none))

Commit message: Update design.
Parts:
- added F1: 自恢复保险丝, Fuse:Fuse_1206_3216Metric, F.Cu at (96.0, 120.9)
- added Q1: S8550, Uinio:SOT-23-3_L2.9-W1.6-P1.90-LS2.9-BL, F.Cu at (98.9, 129.7)
- added R13: 1.5K, Resistor_SMD:R_0603_1608Metric, F.Cu at (109.1, 129.5)
- added R14: 1.5K, Resistor_SMD:R_0603_1608Metric, F.Cu at (109.1, 125.4)
- added R15: 1.5K, Resistor_SMD:R_0603_1608Metric, F.Cu at (107.1, 129.4)
- added R16: 0, Resistor_SMD:R_0603_1608Metric, F.Cu at (107.1, 125.4)
- Y1: footprint Crystal:Crystal_SMD_0603-4Pin_6.0x3.5mm -> Crystal:Crystal_SMD_3225-4Pin_3.2x2.5mm
- moved C4 1.15 mm to (129.0, 99.1)
- moved C3 1.13 mm to (129.0, 102.9)
- moved Y1 1.07 mm to (126.1, 101.0)
Connections:
- J5 pad 5: /_JTAG_nSRST_Output -> /_JTAG_nSRST_Input
- J5 pad 8: /_VDD_3.3V -> /3.3V_Input
- U2 pad 28: /USB_ENUM -> /USB_Enumeration
- USB1 pad A4B9: /VDD_5V -> Net-(USB1-PadA4B9)
Routing:
- net Net-(C4-Pad2): track 1.35 -> 3.27 mm
- net Net-(U2-Pad6): track 7.33 -> 6.38 mm
Other:
- outline, holes or cut-outs redrawn

Commit message: Prepare Version 2.0.0.
Parts:
- removed F1: 自恢复保险丝, Fuse:Fuse_1206_3216Metric
- removed Q1: S8550, Uinio:SOT-23-3_L2.9-W1.6-P1.90-LS2.9-BL
- removed R13, R14, R15: 1.5K, Resistor_SMD:R_0603_1608Metric
- removed R16: 0, Resistor_SMD:R_0603_1608Metric
- moved ? 2.96 mm to (127.3, 107.7), turned to 90 degrees
Connections:
- U2 pad 28: /USB_Enumeration -> unconnected-(U2-Pad28)
- USB1 pad A4B9: Net-(USB1-PadA4B9) -> /VDD_5V
Routing:
- net /_JTAG_nSRST_Output: track 28.6 -> 11.3 mm
- net /_JTAG_nSRST_Input: track 0.00 -> 16.3 mm
- net /3.3V_Input: track 27.4 -> 37.7 mm, vias 3 -> 4
- net GND: track 179.5 -> 181.3 mm, vias 25 -> 26
- net Net-(U2-Pad5): track 6.77 -> 6.07 mm

Commit message: Release UINIO-DAP-Link 2.0.0.
Parts:
- moved ? 0.08 mm to (127.3, 107.6)
Other:
- board text added: "Version 2.0.0"
- board text removed: "Version 1.0.0"
Changed lines of the file:
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@@
   (title_block
     (title "UINIO-DAP-Link")
-    (date "2022-10-26")
-    (rev "Version 1.0.0")
+    (date "2022-11-17")
+    (rev "Version 2.0.0")
     (company "电子技术博客 UinIO.com")
   )
@@
   )
   (footprint "LOGO" (layer "F.Cu")
-    (at 127.29 107.65 90)
+    (at 127.28 107.57 90)
     (attr board_only exclude_from_pos_files exclude_from_bom)
     (fp_text reference "" (at 0 0 90) (layer "F.SilkS")
@@
     (effects (font (size 0.9 0.9) (thickness 0.15)) (justify mirror))
   )
-  (gr_text "Version 1.0.0" (at 104.84 107.47 90) (layer "B.SilkS")
+  (gr_text "Version 2.0.0" (at 104.84 107.47 90) (layer "B.SilkS")
     (effects (font (size 0.7 0.7) (thickness 0.1)) (justify mirror))
   )
@@
     (effects (font (size 1 1) (thickness 0.1)))
   )
+  (gr_text "GND" (at 106.96 113.64 45) (layer "F.SilkS")
+    (effects (font (size 0.7 0.7) (thickness 0.1)))
+  )
   (gr_text "TX" (at 166.88 97.58 270) (layer "F.SilkS")
     (effects (font (size 1 1) (thickness 0.2)))
   )
+  (gr_text "3.3V" (at 114.51 113.5 45) (layer "F.SilkS")
+    (effects (font (size 0.7 0.7) (thickness 0.1)))
+  )
+  (gr_text "SWDIO" (at 112.33 113.15 45) (layer "F.SilkS")
+    (effects (font (size 0.7 0.7) (thickness 0.1)))
+  )
   (gr_text "RX" (at 164.36 97.55 270) (layer "F.SilkS")
     (effects (font (size 1 1) (thickness 0.2)))
   )
+  (gr_text "SWCLK" (at 109.89 113.07 45) (layer "F.SilkS")
+    (effects (font (size 0.7 0.7) (thickness 0.1)))
+  )
   (segment (start 130.07 106.7) (end 128.94 106.7) (width 0.3) (layer "F.Cu") (net 1))

Commit message: Release UINIO-DAP-Link 3.0.0.
Parts:
- removed the ? at (178.8, 107.4)
- removed the ? at (127.3, 107.6)
- added ?: LOGO, LOGO, F.Cu at (128.2, 102.1)
- added ?: LOGO, LOGO, F.Cu at (178.8, 107.3)
- added ?: LOGO, LOGO, F.Cu at (130.4, 103.1)
- added R13: 22R, Resistor_SMD:R_0603_1608Metric, F.Cu at (113.5, 107.3)
- added R14: 22R, Resistor_SMD:R_0603_1608Metric, F.Cu at (113.5, 105.9)
- added R15: 1.5K, Resistor_SMD:R_0603_1608Metric, F.Cu at (113.5, 108.8)
- moved R6 17.4 mm to (124.8, 115.8), turned to -90 degrees
- moved R9 17.1 mm to (121.4, 99.0), turned to -90 degrees
- moved C5 16.8 mm to (123.1, 115.8), turned to -90 degrees
- moved R12 16.6 mm to (119.7, 99.0), turned to 90 degrees
- moved D5 16.5 mm to (118.0, 99.0), turned to -90 degrees
- moved C4 13.0 mm to (130.7, 112.0)
- moved Y1 12.6 mm to (128.2, 113.4)
- moved C3 12.2 mm to (130.7, 115.0)
- moved R11 9.54 mm to (119.7, 115.8)
- moved D4 8.02 mm to (118.0, 115.8)
- moved R7 6.45 mm to (124.9, 99.0)
- moved R8 6.40 mm to (123.2, 99.0)
- moved R10 6.23 mm to (121.4, 115.8)
- moved U2 2.42 mm to (121.4, 107.3), turned to 45 degrees
- moved ? 0.35 mm to (120.8, 107.3), turned to 180 degrees
Connections:
- USB1 pad A6: /USB_Data_P -> /USB_+
- USB1 pad A7: /USB_Data_N -> /USB_-
- USB1 pad B6: /USB_Data_P -> /USB_+
- USB1 pad B7: /USB_Data_N -> /USB_-
Routing:
- net /VDD_3.3V: track 68.5 -> 97.1 mm, vias 6 -> 4
- net /JTAG_TDI: track 26.0 -> 9.39 mm, vias 4 -> 0
- net GND: track 181.3 -> 166.7 mm, vias 26 -> 23
- net /JTAG_TDO: track 18.5 -> 7.92 mm
- net /JTAG_TCK/SWCLK: track 28.6 -> 18.2 mm
- net /USART2_RX: track 18.7 -> 8.46 mm, vias 1 -> 0
- net /USART2_TX: track 18.8 -> 9.16 mm, vias 2 -> 0
- net /JTAG_nTRST: track 24.4 -> 15.9 mm
- net Net-(R9-Pad2): track 11.2 -> 2.96 mm, vias 2 -> 0
- net /Download_SWDIO: track 6.93 -> 13.9 mm, vias 1 -> 2
- net /JTAG_TMS/SWDIO: track 34.5 -> 28.4 mm, vias 2 -> 0
- net /USB_-: track 0.00 -> 5.72 mm
- net /USB_+: track 0.00 -> 5.72 mm
- net /Download_SWCLK: track 15.3 -> 9.87 mm, vias 1 -> 0
- net /USB_Data_N: track 9.92 -> 5.92 mm
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Other:
- board text added: "SWD-JTAG 转接板"
- board text added: "Version 3.0.0"
- board text added: "运行"
- board text added: "连接"
- board text removed: "Version 2.0.0"

Commit message: Release UINIO-DAP-Link version 3.0.1.
Other:
- board text added: "Version 3.0.1"
- board text removed: "Version 3.0.0"
