File: UINIO-DAPLink.kicad_pcb (KiCad board)
At the start: 2 copper layers, 90.4 x 31 mm, 53 parts, among them J1 扩展板串口 & 电源输出, J2 扩展板 JTAG 输出, J3 JTAG_nTRST 跳线选择, J4 3.3V 跳线选择, J5 扩展板 SWD 输入, J6 DAPLink 固件下载接口, J7 SWD 下载输出, U1 ME6211, U2 STM32F103C8T6, Y1 8MHz

Commit message: update
Parts:
- C1: value 10nF -> 1uF; footprint Capacitor_SMD:C_0402_1005Metric -> Capacitor_SMD:C_0603_1608Metric
- C10: value 0.1uF -> 1uF
- C2: value 10uF -> 1uF; footprint Capacitor_SMD:C_0402_1005Metric -> Capacitor_SMD:C_0603_1608Metric
- U1: value ME6211 -> ME6211C33M5G
- moved J6 32.1 mm to (97.2, 146.8)
- moved C5 22.9 mm to (121.6, 152.1)
- moved R6 22.9 mm to (118.6, 152.2)
- moved J5 11.8 mm to (153.4, 119.5)
- moved U1 2.29 mm to (107.1, 127.9)
- moved C1 2.29 mm to (110.6, 128.8)
- moved C2 2.29 mm to (110.6, 126.9)
Connections:
- C1 pad 1: GND -> /VDD_5V
- C1 pad 2: Net-(U1-NC) -> GND
- U1 pad 4: Net-(U1-NC) -> unconnected-(U1-NC-Pad4)

Commit message: update
Parts:
- moved R17 32.9 mm to (104.3, 141.8)
- moved R15 31.5 mm to (109.9, 140.1), turned to 0 degrees
- moved R14 31.4 mm to (106.7, 136.6)
- moved R13 31.0 mm to (106.8, 137.6)
- moved R16 30.6 mm to (104.0, 133.4)
- moved D5 29.6 mm to (124.6, 127.9)
- moved R12 28.9 mm to (126.5, 128.0)
- moved R10 21.0 mm to (110.7, 133.7), turned to 180 degrees
- moved R8 20.7 mm to (128.5, 141.3), turned to 0 degrees
- moved R7 20.5 mm to (128.9, 144.5), turned to 180 degrees
- moved R9 17.6 mm to (128.4, 132.0), turned to 0 degrees
- moved D4 12.6 mm to (115.1, 128.0)
- moved R11 12.6 mm to (116.9, 128.0), turned to 90 degrees
- moved C1 5.02 mm to (105.7, 127.6), turned to -90 degrees
- moved USB1 3.50 mm to (97.5, 136.9)
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Connections:
- J3 pad 1: /_JTAG_nSRST_Input -> /_JTAG_nSRST
- J5 pad 3: /_JTAG_nSRST_Input -> /_JTAG_TDO
- R4 pad 1: /_JTAG_TDO -> /_JTAG_nSRST

Commit message: update
Parts:
- removed ?: LOGO, LOGO
- removed HOLE1, HOLE2: Hole-1mm, Uinio:Hole-1mm
- removed HOLE3, HOLE4, HOLE5, HOLE6, HOLE7, HOLE8: Hole-2mm, Uinio:Hole-2mm
- added HOLE**: Hole-2mm, Uinio:Hole-2mm, F.Cu at (96.0, 126.0)
- added HOLE**: Hole-2mm, Uinio:Hole-2mm, F.Cu at (156.8, 124.4)
- added HOLE**: Hole-2mm, Uinio:Hole-2mm, F.Cu at (174.5, 148.9)
- added HOLE**: Hole-2mm, Uinio:Hole-2mm, F.Cu at (156.8, 148.8)
- added HOLE**: Hole-2mm, Uinio:Hole-2mm, F.Cu at (96.0, 147.4)
- added HOLE**: Hole-2mm, Uinio:Hole-2mm, F.Cu at (132.7, 126.0)
- added HOLE**: Hole-2mm, Uinio:Hole-2mm, F.Cu at (132.7, 147.4)
- added HOLE**: Hole-2mm, Uinio:Hole-2mm, F.Cu at (174.5, 124.5)
- J6: footprint Connector_PinHeader_2.54mm:PinHeader_1x04_P2.54mm_Vertical -> Connector_PinHeader_2.54mm:PinHeader_1x05_P2.54mm_Vertical
- R11, R12: footprint Resistor_SMD:R_0402_1005Metric -> Resistor_SMD:R_0603_1608Metric
- moved J4 30.3 mm to (160.6, 149.9)
- moved J3 30.3 mm to (168.2, 149.9)
- moved R1 29.7 mm to (169.4, 142.0)
- moved R3 29.7 mm to (169.4, 131.7)
- moved R2 29.6 mm to (169.4, 133.8)
- moved D1 29.6 mm to (166.2, 142.0)
- moved R4 29.6 mm to (166.2, 138.9)
- moved R5 29.6 mm to (166.2, 137.1)
- moved D2 29.6 mm to (166.1, 133.8)
- moved D3 29.6 mm to (166.1, 131.7)
- moved J2 29.6 mm to (177.7, 125.2)
- moved J5 28.9 mm to (149.8, 148.1)
- moved J1 28.8 mm to (160.6, 123.5)
- moved J6 24.3 mm to (109.3, 125.8)
- moved D5 18.8 mm to (125.6, 146.7), turned to 90 degrees
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Connections:
- net /_JTAG_nSRST_Output renamed /_JTAG_nRST_Output
- net /nTRST renamed /nRST
- J3 pad 1: /_JTAG_nSRST -> /_JTAG_nRST
- J5 pad 10: /_VDD_5V -> /_VDD_3.3V
- J5 pad 5: Net-(J5-Pin_5) -> /_VDD_5V
- J5 pad 6: GND -> Net-(J5-Pin_6)
- J5 pad 9: /_VDD_3.3V -> GND
- J6 pad 1: GND -> /NRST
- J6 pad 4: /VDD_3.3V -> GND
- J7 pad 10: /VDD_5V -> /VDD_3.3V
- J7 pad 4: /JTAG_nTRST -> /JTAG_TDI
- J7 pad 5: /JTAG_TDI -> /VDD_5V
- J7 pad 6: GND -> /JTAG_nRST
- J7 pad 9: /VDD_3.3V -> GND
- R4 pad 1: /_JTAG_nSRST -> /_JTAG_TDI
- R5 pad 1: /_JTAG_TDI -> /_JTAG_nRST
- R5 pad 2: Net-(J5-Pin_5) -> Net-(J5-Pin_6)
- R7 pad 1: /JTAG_nTRST -> /JTAG_nRST
- U2 pad 18: /JTAG_nTRST -> /JTAG_nRST
Routing:
- net /VDD_3.3V: track 8.67 -> 6.89 mm
Other:
- board size 90.4 x 31 mm -> 95.7 x 30 mm
- board text added: "3V3"
- board text added: "CLK"
- board text added: "DIO"
- board text added: "NRST"
- board text added: "Version 5.0.0"
- board text added: "nRST"
- board text removed: "nTRST"
