File: UINIO-DAPLink.kicad_pcb (KiCad board)
At the start: 2 copper layers, 94 x 30 mm, 52 parts, among them J1 扩展板串口 & 电源输出, J2 扩展板 JTAG 输出, J3 JTAG_nTRST 跳线选择, J4 3.3V 跳线选择, J5 扩展板 SWD 输入, J6 DAPLink 固件下载接口, J7 SWD 下载输出, U1 ME6211C33M5G, U2 STM32F103C8T6, Y1 8MHz

Commit message: update
Parts:
- moved C7 34.5 mm to (116.7, 102.1)
- moved HOLE** 34.5 mm to (102.8, 113.3)
- moved C2 34.5 mm to (112.5, 93.3)
- moved C6 34.5 mm to (125.4, 96.4)
- moved R13 34.5 mm to (109.3, 102.6)
- moved R15 34.5 mm to (112.4, 102.6)
- moved R4 34.5 mm to (173.7, 103.9)
- moved USB1 34.5 mm to (103.5, 102.6)
- moved C1 34.5 mm to (107.2, 93.3)
- moved C10 34.5 mm to (126.9, 113.2)
- moved C3 34.5 mm to (118.8, 112.3)
- moved C8 34.5 mm to (134.7, 102.9)
- moved D1 34.5 mm to (174.3, 96.3)
- moved HOLE** 34.5 mm to (179.8, 114.8)
- moved HOLE** 34.5 mm to (162.2, 114.8)
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Other:
- board size 94 x 30 mm -> 94.1 x 30 mm

Commit message: update
Parts:
- added D6: 1N4007, Diode_SMD:D_SMA, F.Cu at (110.2, 109.4)
- F1: value Fuse -> 60V 1A
- moved F1 13.7 mm to (109.5, 96.2)
- moved R6 2.90 mm to (125.4, 113.1), turned to -90 degrees
- moved C4 1.36 mm to (116.5, 108.1)
- moved C3 1.33 mm to (119.5, 111.2)
- moved Y1 1.16 mm to (118.7, 108.9)
- moved U1 1.10 mm to (109.4, 92.3)
- moved C2 1.10 mm to (112.1, 92.3)
- moved C1 1.10 mm to (106.8, 92.3)
- moved C5 0.16 mm to (123.8, 113.1), turned to -90 degrees
- moved C10 0.13 mm to (127.0, 113.1)
Connections:
- J7 pad 1: /USART2_TX -> unconnected-(J7-Pin_1-Pad1)
Routing:
- net /JTAG_nRST: track 0.00 -> 36.4 mm
- net /USB_Data_N: track 0.00 -> 25.6 mm
- net /USB_Data_P: track 0.00 -> 25.4 mm
- net /USART2_RX: track 0.00 -> 22.7 mm
- net /JTAG_TDI: track 0.00 -> 21.6 mm
- net /JTAG_TDO: track 0.00 -> 21.2 mm
- net /JTAG_TMS/SWDIO: track 0.00 -> 21.1 mm
- net /JTAG_TCK/SWCLK: track 0.00 -> 18.5 mm
- net /VDD_3.3V: track 6.89 -> 25.4 mm, vias 0 -> 3
- net Net-(U2-NRST): track 0.00 -> 9.64 mm
- net Net-(U2-PD1-OSC_OUT): track 0.59 -> 6.94 mm
- net /USB_-: track 0.00 -> 5.99 mm
- net Net-(U2-PB2): track 0.00 -> 5.97 mm
- net Net-(U2-BOOT0): track 0.00 -> 4.86 mm
- net Net-(U2-PD0-OSC_IN): track 0.00 -> 3.98 mm
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- added copper zone on B.Cu, net /VDD_3.3V
- added copper zone on F.Cu, net /VDD_3.3V
- added copper zone on F.Cu, net /VDD_5V
- added copper zone on B.Cu, net GND
- added copper zone on F.Cu, net GND

Commit message: update
Parts:
- turned F1 to 180 degrees
Connections:
- net /_VDD_5V renamed /_VDD_5V_Fuse
- C1 pad 1: /VDD_5V -> /VDD_5V_Fuse
- D6 pad 1: /VDD_5V -> /VDD_5V_Fuse
- F1 pad 1: /VDD_5V -> /VDD_5V_Fuse
- J7 pad 5: /VDD_5V -> /VDD_5V_Fuse
- U1 pad 1: /VDD_5V -> /VDD_5V_Fuse
- U1 pad 3: /VDD_5V -> /VDD_5V_Fuse
Routing:
- net /VDD_5V_Fuse: track 0.00 -> 14.4 mm, vias 0 -> 2
- net /VDD_5V: track 0.01 -> 5.89 mm, vias 0 -> 2
- net GND: track 1.62 -> 5.86 mm
- net /USB_+: track 2.98 -> 4.81 mm, vias 0 -> 2
- net Net-(USB1-CC2): track 3.67 -> 4.20 mm
- added copper zone on F.Cu, net /VDD_5V_Fuse

Commit message: update
Routing:
- net /VDD_5V_Fuse: track 14.4 -> 26.9 mm
- net GND: vias 0 -> 63

Commit message: update
Parts:
- removed R4, R5: 22R, Resistor_SMD:R_0402_1005Metric
- moved HOLE** 0.07 mm to (162.1, 90.4)
- moved HOLE** 0.07 mm to (162.1, 114.8)
Connections:
- C5 pad 1: Net-(U2-NRST) -> /NRST
- J5 pad 4: Net-(J5-Pin_4) -> /_JTAG_TDI
- J5 pad 6: Net-(J5-Pin_6) -> /_JTAG_nRST
- J7 pad 1: unconnected-(J7-Pin_1-Pad1) -> /USART2_TX
- R6 pad 1: Net-(U2-NRST) -> /NRST
- U2 pad 28: unconnected-(U2-PB15-Pad28) -> /USB_ENUM
- U2 pad 7: Net-(U2-NRST) -> /NRST
Routing:
- net Net-(U2-NRST): track 9.48 -> 0.00 mm
- net /NRST: track 0.00 -> 9.48 mm

Commit message: Finish PCB Layout.
Parts:
- J5, J7: footprint Connector_PinHeader_2.54mm:PinHeader_1x10_P2.54mm_Vertical -> Connector_PinSocket_2.54mm:PinSocket_1x11_P2.54mm_Vertical
- moved J1 28.3 mm to (176.0, 115.9), turned to -90 degrees
- moved J3 27.5 mm to (165.9, 89.4)
- moved J4 27.5 mm to (173.5, 89.4)
- moved D5 21.2 mm to (132.6, 91.5), turned to -90 degrees
- moved R12 21.2 mm to (134.1, 91.5), turned to -90 degrees
- moved D4 20.2 mm to (132.6, 112.7), turned to 90 degrees
- moved R11 20.2 mm to (134.1, 112.7), turned to 90 degrees
- moved R15 2.29 mm to (110.4, 103.7)
- moved D3 1.26 mm to (174.3, 107.7)
- moved R3 1.26 mm to (171.1, 107.7)
- moved J5 1.25 mm to (155.1, 115.3)
- moved J7 1.25 mm to (147.5, 115.3)
- moved R2 1.24 mm to (171.1, 110.2)
- moved D2 1.24 mm to (174.3, 110.2)
- moved R14 1.10 mm to (110.4, 101.6)
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Connections:
- J5 pad 1: /_USART2_TX -> /_VDD_5V_Fuse
- J5 pad 10: /_VDD_3.3V -> GND
- J5 pad 2: /_USART2_RX -> GND
- J5 pad 3: /_JTAG_TDO -> /_USART2_TX
- J5 pad 4: /_JTAG_TDI -> /_USART2_RX
- J5 pad 5: /_VDD_5V_Fuse -> /_JTAG_TDO
- J5 pad 6: /_JTAG_nRST -> /_JTAG_TDI
- J5 pad 7: /_JTAG_TCK/SWCLK -> /_JTAG_nRST
- J5 pad 8: /_JTAG_TMS/SWDIO -> /_JTAG_TCK/SWCLK
- J5 pad 9: GND -> /_JTAG_TMS/SWDIO
- J7 pad 1: /USART2_TX -> /VDD_5V_Fuse
- J7 pad 10: /VDD_3.3V -> GND
- J7 pad 2: /USART2_RX -> GND
- J7 pad 3: /JTAG_TDO -> /USART2_TX
- J7 pad 4: /JTAG_TDI -> /USART2_RX
- J7 pad 5: /VDD_5V_Fuse -> /JTAG_TDO
- J7 pad 6: /JTAG_nRST -> /JTAG_TDI
- J7 pad 7: /JTAG_TCK/SWCLK -> /JTAG_nRST
- J7 pad 8: /JTAG_TMS/SWDIO -> /JTAG_TCK/SWCLK
- J7 pad 9: GND -> /JTAG_TMS/SWDIO
Routing:
- net /VDD_3.3V: track 25.4 -> 62.3 mm, vias 3 -> 8
- net /_JTAG_TDI: track 0.00 -> 30.5 mm, vias 0 -> 1
- net /_JTAG_TMS/SWDIO: track 0.00 -> 29.5 mm
- net /_JTAG_TCK/SWCLK: track 0.00 -> 29.5 mm
- net /_JTAG_TDO: track 0.00 -> 28.4 mm
- net /_VDD_3.3V: track 0.00 -> 27.8 mm
- net /_JTAG_nRST_Output: track 0.00 -> 27.0 mm
- net /VDD_5V_Fuse: track 26.9 -> 0.04 mm, vias 2 -> 8
- net /_USART2_RX: track 0.00 -> 25.9 mm
- net /USART2_TX: track 0.00 -> 24.3 mm
- net /_USART2_TX: track 0.00 -> 22.2 mm
- net Net-(D4-A): track 0.00 -> 18.8 mm, vias 0 -> 2
- net /NRST: track 9.48 -> 27.7 mm, vias 0 -> 1
- net /Download_SWDIO: track 0.00 -> 11.1 mm, vias 0 -> 1
- net /JTAG_nRST: track 36.4 -> 25.4 mm
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- added copper zone on B.Cu, net /VDD_5V_Fuse
Other:
- outline, holes or cut-outs redrawn
- board text added: "JTAG接口 3.3V跳线"
- board text added: "JTAG接口 nSRST跳线"
- board text removed: "3.3V跳线"
- board text removed: "JTAG接口"
- board text removed: "nSRST跳线"
