File: UINIO-DAPLink.kicad_sch (KiCad schematic)
At the start: 44 parts, among them J1 扩展板串口 & 电源输出, J2 扩展板 JTAG 输出, J3 JTAG_nTRST 跳线选择, J4 3.3V 跳线选择, J5 扩展板 SWD 输入, J6 DAPLink 固件下载接口, J7 SWD 下载输出, U1 ME6211, U2 STM32F103C8T6, Y1 8MHz

Commit message: update
Parts:
- C1: value 10nF -> 1uF; footprint Capacitor_SMD:C_0402_1005Metric -> Capacitor_SMD:C_0603_1608Metric
- C10: value 0.1uF -> 1uF
- C2: value 10uF -> 1uF; footprint Capacitor_SMD:C_0402_1005Metric -> Capacitor_SMD:C_0603_1608Metric
- U1: value ME6211 -> ME6211C33M5G
Connections:
- net GND: now also C1.2; no longer C1.1
- net VDD_5V: now also C1.1
- net at U1.4 (NC): no longer C1.2
- no-connect marks 26 -> 27
Other:
- moved on the sheet: C2, U1

Commit message: update
Connections:
- net _JTAG_TDO: now also J5.3 (Pin_3); no longer R4.1
- net _JTAG_nSRST_Input renamed _JTAG_nSRST
- net _JTAG_nSRST: now also R4.1; no longer J5.3 (Pin_3)
Changed lines of the file:
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@@
 		)
 	)
-	(label "_JTAG_nSRST_Input"
-		(at 120.65 173.99 0)
+	(label "_JTAG_nSRST"
+		(at 120.65 176.53 0)
 		(fields_autoplaced yes)
 		(effects
@@
 		)
 	)
-	(label "_JTAG_nSRST_Input"
+	(label "_JTAG_nSRST"
 		(at 68.58 181.61 0)
 		(fields_autoplaced yes)
@@
 	)
 	(label "_JTAG_TDO"
-		(at 120.65 176.53 0)
-		(fields_autoplaced yes)
-		(effects
+		(at 120.65 173.99 0)
+		(fields_autoplaced yes)
+		(effects

Commit message: update
Parts:
- removed J6: DAPLink 固件下载接口, Connector_PinHeader_2.54mm:PinHeader_1x04_P2.54mm_Vertical, symbol Connector:Conn_01x04_Pin
- added J6: DAPLink 固件下载接口, Connector_PinHeader_2.54mm:PinHeader_1x05_P2.54mm_Vertical, symbol Connector:Conn_01x05_Pin
- R11, R12: footprint Resistor_SMD:R_0402_1005Metric -> Resistor_SMD:R_0603_1608Metric
Connections:
- net Download_SWCLK: now also J6.2 (Pin_2)
- net Download_SWDIO: now also J6.3 (Pin_3)
- net GND: now also J5.9 (Pin_9), J7.9 (Pin_9), J6.4 (Pin_4); no longer J5.6 (Pin_6), J7.6 (Pin_6)
- net JTAG_TDI: now also J7.4 (Pin_4); no longer J7.5 (Pin_5)
- net VDD_3.3V: now also J7.10 (Pin_10), J6.5 (Pin_5); no longer J7.9 (Pin_9)
- net VDD_5V: now also J7.5 (Pin_5); no longer J7.10 (Pin_10)
- net _JTAG_TDI: now also R4.1; no longer R5.1
- net _VDD_3.3V: now also J5.10 (Pin_10); no longer J5.9 (Pin_9)
- net _VDD_5V: now also J5.5 (Pin_5); no longer J5.10 (Pin_10)
- net at R5.2: now also J5.6 (Pin_6); no longer J5.5 (Pin_5)
- net JTAG_nTRST renamed JTAG_nRST
- net JTAG_nRST: now also J7.6 (Pin_6); no longer J7.4 (Pin_4)
- net _JTAG_nSRST renamed _JTAG_nRST
- net _JTAG_nRST: now also R5.1; no longer R4.1
- net _JTAG_nSRST_Output renamed _JTAG_nRST_Output
- net nTRST renamed nRST
- new net NRST: J6.1 (Pin_1)
Other:
- moved on the sheet: D1, R1, R5
