File: UINIO-DAPLink.kicad_sch (KiCad schematic)
At the start: 44 parts, among them J1 扩展板串口 & 电源输出, J2 扩展板 JTAG 输出, J3 JTAG_nTRST 跳线选择, J4 3.3V 跳线选择, J5 扩展板 SWD 输入, J6 DAPLink 固件下载接口, J7 SWD 下载输出, U1 ME6211C33M5G, U2 STM32F103C8T6, Y1 8MHz

Commit message: update
Other:
- note added: "ME6211C33M5G 线性稳压器"
- note added: "SWD-JTAG 转接板"
- note removed: "JTAG 扩展板"
- note removed: "ME6211 线性稳压器"
Changed lines of the file:
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@@
 		)
 	)
-	(text "JTAG 扩展板"
+	(text "SWD-JTAG\n转接板"
 		(exclude_from_sim no)
-		(at 74.168 149.86 0)
+		(at 92.964 151.892 0)
 		(effects
 			(font
 				(size 4 4)
 			)
-			(justify left bottom)
+			(justify bottom)
 		)
 	)
@@
 		)
 	)
-	(text "ME6211 线性稳压器\n"
+	(text "ME6211C33M5G 线性稳压器\n"
 		(exclude_from_sim no)
-		(at 39.37 57.912 0)
+		(at 30.48 57.912 0)
 		(effects
 			(font

Commit message: update
Parts:
- added D6: 1N4007, Diode_THT:D_DO-41_SOD81_P10.16mm_Horizontal, symbol Diode:1N4007
- F1: value Fuse -> 60V 1A
Connections:
- net GND: now also D6.2 (A)
- net USART2_TX: no longer J7.1 (Pin_1)
- net VDD_5V: now also D6.1 (K)
Other:
- note added: "过流 & 防反接"
- moved on the sheet: F1, J6, J7, R13, R14, R15, R16, R17, USB1

Commit message: update
Parts:
- D6: footprint Diode_THT:D_DO-41_SOD81_P10.16mm_Horizontal -> Diode_SMD:D_SMA
Other:
- moved on the sheet: D6, F1
Changed lines of the file:
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@@
 	)
 	(junction
-		(at 132.08 31.75)
+		(at 143.51 31.75)
 		(diameter 0)
 		(color 0 0 0 0)
@@
 	(wire
 		(pts
-			(xy 143.51 31.75) (xy 142.24 31.75)
+			(xy 132.08 31.75) (xy 133.35 31.75)
 		)
 		(stroke
@@
 	(wire
 		(pts
-			(xy 134.62 39.37) (xy 132.08 39.37)
+			(xy 140.97 39.37) (xy 143.51 39.37)
 		)
 		(stroke
@@
 	(wire
 		(pts
-			(xy 132.08 39.37) (xy 132.08 31.75)
+			(xy 143.51 39.37) (xy 143.51 31.75)
 		)
 		(stroke
@@
 	(wire
 		(pts
-			(xy 129.54 31.75) (xy 132.08 31.75)
+			(xy 146.05 31.75) (xy 143.51 31.75)
 		)
 		(stroke
@@
 	(wire
 		(pts
-			(xy 132.08 31.75) (xy 134.62 31.75)
+			(xy 143.51 31.75) (xy 140.97 31.75)
 		)
 		(stroke
@@
 	(wire
 		(pts
-			(xy 142.24 39.37) (xy 143.51 39.37)
+			(xy 133.35 39.37) (xy 132.08 39.37)
 		)
 		(stroke
@@
 	)
 	(label "VDD_5V"
-		(at 143.51 31.75 0)
+		(at 132.08 31.75 180)
 		(fields_autoplaced yes)
 		(effects
@@
 				(size 1.27 1.27)
 			)
-			(justify left bottom)
+			(justify right bottom)
 		)
 	)
@@
 	)
 	(label "VDD_5V"
-		(at 129.54 31.75 180)
+		(at 146.05 31.75 0)
 		(fields_autoplaced yes)
 		(effects
@@
 				(size 1.27 1.27)
 			)
-			(justify right bottom)
+			(justify left bottom)
 		)
 	)
@@
 	(symbol
 		(lib_id "power:GND")
-		(at 143.51 39.37 90)
-		(mirror x)
+		(at 132.08 39.37 270)
 		(unit 1)
 		(exclude_from_sim no)
@@
 		(dnp no)
 		(property "Reference" "#PWR030"
-			(at 149.86 39.37 0)
+			(at 125.73 39.37 0)
 			(effects
 				(font
@@
 		)
 		(property "Value" "GND"
-			(at 146.304 39.37 90)
+			(at 129.286 39.37 90)
 			(effects
 				(font
@@
 		)
 		(property "Footprint" ""
-			(at 143.51 39.37 0)
+			(at 132.08 39.37 0)
 			(effects
 				(font
@@
 		)
 		(property "Datasheet" ""
-			(at 143.51 39.37 0)
+			(at 132.08 39.37 0)
 			(effects
 				(font
@@
 		)
 		(property "Description" "Power symbol creates a global label with name \"GND\" , ground"
-			(at 143.51 39.37 0)
+			(at 132.08 39.37 0)
 			(effects
 				(font
@@
 	(symbol
 		(lib_id "Diode:1N4007")
-		(at 138.43 39.37 0)
+		(at 137.16 39.37 0)
+		(mirror y)
 		(unit 1)
 		(exclude_from_sim no)
@@
 		(dnp no)
 		(property "Reference" "D6"
-			(at 141.224 38.354 0)
+			(at 134.366 38.354 0)
 			(effects
 				(font
@@
 		)
 		(property "Value" "1N4007"
-			(at 138.684 42.164 0)
+			(at 136.906 42.164 0)
 			(effects
 				(font
@@
 			)
 		)
-		(property "Footprint" "Diode_THT:D_DO-41_SOD81_P10.16mm_Horizontal"
-			(at 138.43 43.815 0)
+		(property "Footprint" "Diode_SMD:D_SMA"
+			(at 137.16 43.815 0)
 			(effects
 				(font
@@
 		)
 		(property "Datasheet" "http://www.vishay.com/docs/88503/1n4001.pdf"
-			(at 138.43 39.37 0)
+			(at 137.16 39.37 0)
 			(effects
 				(font
@@
 		)
 		(property "Description" "1000V 1A General Purpose Rectifier Diode, DO-41"
-			(at 138.43 39.37 0)
+			(at 137.16 39.37 0)
 			(effects
 				(font
@@
 		)
 		(property "Sim.Device" "D"
-			(at 138.43 39.37 0)
+			(at 137.16 39.37 0)
 			(effects
 				(font
@@
 		)
 		(property "Sim.Pins" "1=K 2=A"
-			(at 138.43 39.37 0)
+			(at 137.16 39.37 0)
 			(effects
 				(font
@@
 	(symbol
 		(lib_id "Device:Fuse")
-		(at 138.43 31.75 90)
+		(at 137.16 31.75 270)
+		(mirror x)
 		(unit 1)
 		(exclude_from_sim no)
@@
 		(dnp no)
 		(property "Reference" "F1"
-			(at 138.43 29.972 90)
+			(at 137.16 29.972 90)
 			(effects
 				(font
@@
 		)
 		(property "Value" "60V 1A"
-			(at 138.43 33.782 90)
+			(at 137.16 33.782 90)
 			(effects
 				(font
@@
 		)
 		(property "Footprint" "Fuse:Fuse_1206_3216Metric"
-			(at 138.43 33.528 90)
+			(at 137.16 33.528 90)
 			(effects
 				(font
@@
 		)
 		(property "Datasheet" "~"
-			(at 138.43 31.75 0)
+			(at 137.16 31.75 0)
 			(effects
 				(font
@@
 		)
 		(property "Description" "Fuse"
-			(at 138.43 31.75 0)
+			(at 137.16 31.75 0)
 			(effects
 				(font

Commit message: update
Connections:
- net VDD_5V: no longer C1.1, D6.1 (K), F1.1, J7.5 (Pin_5), U1.1 (Vin), U1.3 (CE)
- net _VDD_5V renamed _VDD_5V_Fuse
- new net VDD_5V_Fuse: C1.1, D6.1 (K), F1.1, J7.5 (Pin_5), U1.1 (Vin), U1.3 (CE)
Other:
- moved on the sheet: D6, F1
Changed lines of the file:
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@@
 	)
 	(junction
-		(at 143.51 31.75)
+		(at 142.24 31.75)
 		(diameter 0)
 		(color 0 0 0 0)
@@
 	(wire
 		(pts
-			(xy 57.15 95.25) (xy 69.85 95.25)
+			(xy 57.15 95.25) (xy 71.12 95.25)
 		)
 		(stroke
@@
 	(wire
 		(pts
-			(xy 132.08 31.75) (xy 133.35 31.75)
+			(xy 129.54 31.75) (xy 132.08 31.75)
 		)
 		(stroke
@@
 	(wire
 		(pts
-			(xy 140.97 39.37) (xy 143.51 39.37)
+			(xy 139.7 39.37) (xy 142.24 39.37)
 		)
 		(stroke
@@
 	(wire
 		(pts
-			(xy 143.51 39.37) (xy 143.51 31.75)
+			(xy 142.24 39.37) (xy 142.24 31.75)
 		)
 		(stroke
@@
 	(wire
 		(pts
-			(xy 146.05 31.75) (xy 143.51 31.75)
+			(xy 144.78 31.75) (xy 142.24 31.75)
 		)
 		(stroke
@@
 	(wire
 		(pts
-			(xy 143.51 31.75) (xy 140.97 31.75)
+			(xy 142.24 31.75) (xy 139.7 31.75)
 		)
 		(stroke
@@
 	(wire
 		(pts
-			(xy 133.35 39.37) (xy 132.08 39.37)
+			(xy 132.08 39.37) (xy 130.81 39.37)
 		)
 		(stroke
@@
 	(wire
 		(pts
-			(xy 109.22 179.07) (xy 100.33 179.07)
+			(xy 120.65 179.07) (xy 100.33 179.07)
 		)
 		(stroke
@@
 		)
 	)
-	(label "_VDD_5V"
-		(at 109.22 179.07 0)
+	(label "_VDD_5V_Fuse"
+		(at 120.65 179.07 0)
 		(fields_autoplaced yes)
 		(effects
@@
 		)
 	)
-	(label "_VDD_5V"
+	(label "_VDD_5V_Fuse"
 		(at 44.45 184.15 0)
 		(fields_autoplaced yes)
@@
 		)
 	)
-	(label "VDD_5V"
+	(label "VDD_5V_Fuse"
 		(at 36.83 38.1 180)
 		(fields_autoplaced yes)
@@
 		)
 	)
-	(label "VDD_5V"
+	(label "VDD_5V_Fuse"
 		(at 248.92 33.02 0)
 		(fields_autoplaced yes)
@@
 	)
 	(label "VDD_5V"
-		(at 132.08 31.75 180)
+		(at 129.54 31.75 180)
 		(fields_autoplaced yes)
 		(effects
@@
 		)
 	)
-	(label "VDD_5V"
-		(at 146.05 31.75 0)
+	(label "VDD_5V_Fuse"
+		(at 144.78 31.75 0)
 		(fields_autoplaced yes)
 		(effects
@@
 	)
 	(label "VDD_5V"
-		(at 69.85 95.25 0)
+		(at 71.12 95.25 0)
 		(fields_autoplaced yes)
 		(effects
@@
 	(symbol
 		(lib_id "power:GND")
-		(at 132.08 39.37 270)
+		(at 130.81 39.37 270)
 		(unit 1)
 		(exclude_from_sim no)
@@
 		(dnp no)
 		(property "Reference" "#PWR030"
-			(at 125.73 39.37 0)
+			(at 124.46 39.37 0)
 			(effects
 				(font
@@
 		)
 		(property "Value" "GND"
-			(at 129.286 39.37 90)
+			(at 128.016 39.37 90)
 			(effects
 				(font
@@
 		)
 		(property "Footprint" ""
-			(at 132.08 39.37 0)
+			(at 130.81 39.37 0)
 			(effects
 				(font
@@
 		)
 		(property "Datasheet" ""
-			(at 132.08 39.37 0)
+			(at 130.81 39.37 0)
 			(effects
 				(font
@@
 		)
 		(property "Description" "Power symbol creates a global label with name \"GND\" , ground"
-			(at 132.08 39.37 0)
+			(at 130.81 39.37 0)
 			(effects
 				(font
@@
 	(symbol
 		(lib_id "Diode:1N4007")
-		(at 137.16 39.37 0)
+		(at 135.89 39.37 0)
 		(mirror y)
 		(unit 1)
@@
 		(dnp no)
 		(property "Reference" "D6"
-			(at 134.366 38.354 0)
+			(at 133.096 38.354 0)
 			(effects
 				(font
@@
 		)
 		(property "Value" "1N4007"
-			(at 136.906 42.164 0)
+			(at 135.636 42.164 0)
 			(effects
 				(font
@@
 		)
 		(property "Footprint" "Diode_SMD:D_SMA"
-			(at 137.16 43.815 0)
+			(at 135.89 43.815 0)
 			(effects
 				(font
@@
 		)
 		(property "Datasheet" "http://www.vishay.com/docs/88503/1n4001.pdf"
-			(at 137.16 39.37 0)
+			(at 135.89 39.37 0)
 			(effects
 				(font
@@
 		)
 		(property "Description" "1000V 1A General Purpose Rectifier Diode, DO-41"
-			(at 137.16 39.37 0)
+			(at 135.89 39.37 0)
 			(effects
 				(font
@@
 		)
 		(property "Sim.Device" "D"
-			(at 137.16 39.37 0)
+			(at 135.89 39.37 0)
 			(effects
 				(font
@@
 		)
 		(property "Sim.Pins" "1=K 2=A"
-			(at 137.16 39.37 0)
+			(at 135.89 39.37 0)
 			(effects
 				(font
@@
 	(symbol
 		(lib_id "Device:Fuse")
-		(at 137.16 31.75 270)
+		(at 135.89 31.75 270)
 		(mirror x)
 		(unit 1)
@@
 		(dnp no)
 		(property "Reference" "F1"
-			(at 137.16 29.972 90)
+			(at 135.89 29.972 90)
 			(effects
 				(font
@@
 		)
 		(property "Value" "60V 1A"
-			(at 137.16 33.782 90)
+			(at 135.89 33.782 90)
 			(effects
 				(font
@@
 		)
 		(property "Footprint" "Fuse:Fuse_1206_3216Metric"
-			(at 137.16 33.528 90)
+			(at 135.89 33.528 90)
 			(effects
 				(font
@@
 		)
 		(property "Datasheet" "~"
-			(at 137.16 31.75 0)
+			(at 135.89 31.75 0)
 			(effects
 				(font
@@
 		)
 		(property "Description" "Fuse"
-			(at 137.16 31.75 0)
+			(at 135.89 31.75 0)
 			(effects
 				(font

Commit message: update
Connections:
- net USB_ENUM: now reaches U2.28 (PB15)
- no-connect marks 27 -> 26
Other:
- moved on the sheet: C10
Changed lines of the file:
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@@
 	)
 	(junction
-		(at 257.81 134.62)
+		(at 93.98 33.02)
 		(diameter 0)
 		(color 0 0 0 0)
 	)
 	(junction
-		(at 93.98 33.02)
+		(at 40.64 38.1)
 		(diameter 0)
 		(color 0 0 0 0)
 	)
 	(junction
-		(at 40.64 38.1)
+		(at 172.72 119.38)
 		(diameter 0)
 		(color 0 0 0 0)
 	)
 	(junction
-		(at 172.72 119.38)
+		(at 256.54 134.62)
 		(diameter 0)
 		(color 0 0 0 0)
@@
 	)
 	(junction
-		(at 170.18 96.52)
+		(at 172.72 96.52)
 		(diameter 0)
 		(color 0 0 0 0)
@@
 	)
 	(no_connect
-		(at 256.54 127)
-	)
-	(no_connect
 		(at 31.75 140.97)
 	)
@@
 	(wire
 		(pts
+			(xy 256.54 134.62) (xy 259.08 134.62)
+		)
+		(stroke
+			(width 0)
+			(type default)
+		)
+	)
+	(wire
+		(pts
 			(xy 248.92 33.02) (xy 247.65 33.02)
 		)
@@
 	(wire
 		(pts
-			(xy 257.81 134.62) (xy 259.08 134.62)
-		)
-		(stroke
-			(width 0)
-			(type default)
-		)
-	)
-	(wire
-		(pts
 			(xy 140.97 171.45) (xy 157.48 171.45)
 		)
@@
 	(wire
 		(pts
-			(xy 182.88 134.62) (xy 186.69 134.62)
+			(xy 176.53 134.62) (xy 186.69 134.62)
 		)
 		(stroke
@@
 	(wire
 		(pts
-			(xy 236.22 129.54) (xy 257.81 129.54)
+			(xy 236.22 129.54) (xy 256.54 129.54)
 		)
 		(stroke
@@
 	(wire
 		(pts
+			(xy 172.72 96.52) (xy 193.04 96.52)
+		)
+		(stroke
+			(width 0)
+			(type default)
+		)
+	)
+	(wire
+		(pts
 			(xy 83.82 102.87) (xy 83.82 87.63)
 		)
@@
 	(wire
 		(pts
-			(xy 257.81 129.54) (xy 257.81 134.62)
-		)
-		(stroke
-			(width 0)
-			(type default)
-		)
-	)
-	(wire
-		(pts
-			(xy 170.18 96.52) (xy 193.04 96.52)
+			(xy 256.54 129.54) (xy 256.54 134.62)
 		)
 		(stroke
@@
 	(wire
 		(pts
-			(xy 168.91 96.52) (xy 170.18 96.52)
+			(xy 168.91 96.52) (xy 172.72 96.52)
 		)
 		(stroke
@@
 	(wire
 		(pts
-			(xy 251.46 134.62) (xy 257.81 134.62)
+			(xy 251.46 134.62) (xy 256.54 134.62)
 		)
 		(stroke
@@
 	(wire
 		(pts
-			(xy 170.18 96.52) (xy 170.18 97.79)
+			(xy 172.72 96.52) (xy 172.72 97.79)
 		)
 		(stroke
@@
 	)
 	(label "VDD_3.3V"
-		(at 182.88 134.62 180)
+		(at 176.53 134.62 180)
 		(fields_autoplaced yes)
 		(effects
@@
 		)
 	)
+	(label "USB_ENUM"
+		(at 256.54 127 0)
+		(fields_autoplaced yes)
+		(effects
+			(font
+				(size 1.27 1.27)
+			)
+			(justify left bottom)
+		)
+	)
 	(label "VDD_3.3V"
 		(at 172.72 76.2 180)
@@
 	(symbol
 		(lib_id "Device:C")
-		(at 170.18 101.6 0)
+		(at 172.72 101.6 0)
 		(unit 1)
 		(exclude_from_sim no)
@@
 		(dnp no)
 		(property "Reference" "C10"
-			(at 172.466 104.394 0)
+			(at 175.006 104.394 0)
 			(effects
 				(font
@@
 		)
 		(property "Value" "1uF"
-			(at 173.228 99.568 0)
+			(at 175.768 99.568 0)
 			(effects
 				(font
@@
 		)
 		(property "Footprint" "Capacitor_SMD:C_0402_1005Metric"
-			(at 171.1452 105.41 0)
+			(at 173.6852 105.41 0)
 			(effects
 				(font
@@
 		)
 		(property "Datasheet" "~"
-			(at 170.18 101.6 0)
+			(at 172.72 101.6 0)
 			(effects
 				(font
@@
 		)
 		(property "Description" ""
-			(at 170.18 101.6 0)
+			(at 172.72 101.6 0)
 			(effects
 				(font
@@
 	(symbol
 		(lib_id "power:GND")
-		(at 170.18 105.41 0)
+		(at 172.72 105.41 0)
 		(unit 1)
 		(exclude_from_sim no)
@@
 		(dnp no)
 		(property "Reference" "#PWR029"
-			(at 170.18 111.76 0)
+			(at 172.72 111.76 0)
 			(effects
 				(font
@@
 		)
 		(property "Value" "GND"
-			(at 165.1 107.696 0)
+			(at 167.64 107.696 0)
 			(effects
 				(font
@@
 		)
 		(property "Footprint" ""
-			(at 170.18 105.41 0)
+			(at 172.72 105.41 0)
 			(effects
 				(font
@@
 		)
 		(property "Datasheet" ""
-			(at 170.18 105.41 0)
+			(at 172.72 105.41 0)
 			(effects
 				(font
@@
 		)
 		(property "Description" "Power symbol creates a global label with name \"GND\" , ground"
-			(at 170.18 105.41 0)
+			(at 172.72 105.41 0)
 			(effects
 				(font

Commit message: update
Connections:
- net USART2_TX: now also J7.1 (Pin_1)
Changed lines of the file:
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@@
 	(wire
 		(pts
-			(xy 245.11 22.86) (xy 243.84 22.86)
+			(xy 248.92 22.86) (xy 247.65 22.86)
 		)
 		(stroke

Commit message: update
Parts:
- removed R4, R5: 22R, Resistor_SMD:R_0402_1005Metric, symbol Device:R
Connections:
- net NRST: now also C5.1, R6.1, U2.7 (NRST)
- net _JTAG_TDI: now also J5.4 (Pin_4)
- net _JTAG_nRST: now also J5.6 (Pin_6)
- no-connect marks 26 -> 27
Other:
- moved on the sheet: J3, J4

Commit message: Finish PCB Layout.
Parts:
- removed J5: 扩展板 SWD 输入, Connector_PinHeader_2.54mm:PinHeader_1x10_P2.54mm_Vertical, symbol Connector:Conn_01x10_Pin
- removed J7: SWD 下载输出, Connector_PinHeader_2.54mm:PinHeader_1x10_P2.54mm_Vertical, symbol Connector:Conn_01x10_Pin
- added J5: 扩展板 SWD 输入, Connector_PinSocket_2.54mm:PinSocket_1x11_P2.54mm_Vertical, symbol Connector:Conn_01x11_Pin
- added J7: SWD 下载输出, Connector_PinSocket_2.54mm:PinSocket_1x11_P2.54mm_Vertical, symbol Connector:Conn_01x11_Pin
Connections:
- net GND: now also J5.10 (Pin_10), J5.2 (Pin_2), J7.10 (Pin_10), J7.2 (Pin_2)
- net JTAG_TCK/SWCLK: now also J7.8 (Pin_8)
- net JTAG_TDI: now also J7.6 (Pin_6)
- net JTAG_TDO: now also J7.5 (Pin_5)
- net JTAG_TMS/SWDIO: now also J7.9 (Pin_9)
- net JTAG_nRST: now also J7.7 (Pin_7)
- net USART2_RX: now also J7.4 (Pin_4)
- net USART2_TX: now also J7.3 (Pin_3)
- net VDD_3.3V: now also J7.11 (Pin_11)
- net VDD_5V_Fuse: now also J7.1 (Pin_1)
- net _JTAG_TCK/SWCLK: now also J5.8 (Pin_8)
- net _JTAG_TDI: now also J5.6 (Pin_6)
- net _JTAG_TDO: now also J5.5 (Pin_5)
- net _JTAG_TMS/SWDIO: now also J5.9 (Pin_9)
- net _JTAG_nRST: now also J5.7 (Pin_7)
- net _USART2_RX: now also J5.4 (Pin_4)
- net _USART2_TX: now also J5.3 (Pin_3)
- net _VDD_3.3V: now also J5.11 (Pin_11)
- net _VDD_5V_Fuse: now also J5.1 (Pin_1)
Other:
- moved on the sheet: D2, D3, R2, R3
