File: UINIO-DAPLink.kicad_sch (KiCad schematic)
At the start: 43 parts, among them J1 扩展板串口 & 电源输出, J2 扩展板 JTAG 输出, J3 JTAG_nTRST 跳线选择, J4 3.3V 跳线选择, J5 扩展板 SWD 输入, J6 DAPLink 固件下载接口, J7 SWD 下载输出, U1 ME6211C33M5G, U2 STM32F103C8T6, Y1 8MHz

Commit message: Finish PCB Layout.
Parts:
- added D7, D8: LESD5D5.0CT1G, Diode_SMD:D_SOD-523, symbol Diode:1N630xCA
Connections:
- net GND: now also D7.1 (A1), D8.1 (A1); no longer J1.4 (Pin_4), J2.10 (Pin_10), J2.12 (Pin_12), J2.14 (Pin_14), J2.16 (Pin_16), J2.18 (Pin_18), J2.20 (Pin_20), J2.4 (Pin_4), J2.6 (Pin_6), J2.8 (Pin_8), J5.10 (Pin_10), J5.2 (Pin_2), R1.1
- net USB_Data_N: now also D8.2 (A2)
- net USB_Data_P: now also D7.2 (A2)
- new net _GND: J1.4 (Pin_4), J2.10 (Pin_10), J2.12 (Pin_12), J2.14 (Pin_14), J2.16 (Pin_16), J2.18 (Pin_18), J2.20 (Pin_20), J2.4 (Pin_4), J2.6 (Pin_6), J2.8 (Pin_8), J5.10 (Pin_10), J5.2 (Pin_2), R1.1
Other:
- moved on the sheet: R13, R14, R15, R16, R17, USB1

Commit message: Release UINIO-DAPLink version 5.0.0.
Connections:
- net RTCK renamed _JTAG_RTCK
- net nRST renamed _JTAG_TRST
Other:
- moved on the sheet: D7, D8, J1, J3, J4, R13, R14, R15, R16, R17, USB1
